File: Kicad/PixelBytesHost/BatteryCharger.kicad_sch (KiCad schematic)
At the start: 27 parts, among them IC2 TC1108-2.8VDBTR, IC3 TPS61085TDGKR, J2 Type - C, J3 B2B-XH-2__LF__SN_, Q3 SMMBT5551LT1G

Commit message: Demo binary for the board
Connections:
- net 5V: now also Q3.2; no longer C21.2, D1.1 (K), R29.1
- net BAT+: no longer J3.1
- net C_BAT+: now also J3.1
- net In_Vcc: now also IC3.3 (EN); no longer Q3.3
- net display_enable: no longer IC3.3 (EN), Q3.2
- new net display_supply: C21.2, D1.1 (K), Q3.3, R29.1
Changed lines of the file:
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@@
+	)
+	(junction
+		(at 196.85 105.41)
+		(diameter 0)
+		(color 0 0 0 0)
 	)
 	(junction
@@
 	(wire
 		(pts
-			(xy 213.36 161.29) (xy 217.17 161.29)
-		)
-		(stroke
-			(width 0)
-			(type default)
-		)
-	)
-	(wire
-		(pts
 			(xy 100.33 45.72) (xy 115.57 45.72)
 		)
@@
 	(wire
 		(pts
-			(xy 201.93 105.41) (xy 201.93 115.57)
-		)
-		(stroke
-			(width 0)
-			(type default)
-		)
-	)
-	(wire
-		(pts
 			(xy 69.85 48.26) (xy 48.26 48.26)
 		)
@@
 	(wire
 		(pts
+			(xy 213.36 161.29) (xy 215.9 161.29)
+		)
+		(stroke
+			(width 0)
+			(type default)
+		)
+	)
+	(wire
+		(pts
 			(xy 101.6 68.58) (xy 106.68 68.58)
 		)
@@
 	(wire
 		(pts
+			(xy 95.25 124.46) (xy 95.25 128.27)
+		)
+		(stroke
+			(width 0)
+			(type default)
+		)
+	)
+	(wire
+		(pts
 			(xy 62.23 116.84) (xy 62.23 120.65)
 		)
@@
 	(wire
 		(pts
-			(xy 204.47 105.41) (xy 201.93 105.41)
-		)
-		(stroke
-			(width 0)
-			(type default)
-		)
-	)
-	(wire
-		(pts
 			(xy 128.27 180.34) (xy 128.27 184.15)
 		)
@@
 		(pts
 			(xy 219.71 48.26) (xy 223.52 48.26)
+		)
+		(stroke
+			(width 0)
+			(type default)
+		)
+	)
+	(wire
+		(pts
+			(xy 196.85 105.41) (xy 204.47 105.41)
 		)
 		(stroke
@@
 		)
 	)
-	(global_label "display_enable"
-		(shape input)
-		(at 201.93 115.57 270)
-		(effects
-			(font
-				(size 1.27 1.27)
-			)
-			(justify right)
-		)
-		(property "Intersheetrefs" "${INTERSHEET_REFS}"
-			(at 201.93 115.57 0)
-			(effects
-				(font
-					(size 1.27 1.27)
-				)
-				(hide yes)
-			)
-		)
-	)
-	(global_label "BAT+"
-		(shape input)
-		(at 217.17 161.29 0)
-		(effects
-			(font
-				(size 1.27 1.27)
-			)
-			(justify left)
-		)
-		(property "Intersheetrefs" "${INTERSHEET_REFS}"
-			(at 217.17 161.29 0)
-			(effects
-				(font
-					(size 1.27 1.27)
-				)
-				(hide yes)
-			)
-		)
-	)
 	(global_label "C_BAT+"
 		(shape input)
-		(at 121.92 50.8 0)
+		(at 215.9 161.29 0)
 		(fields_autoplaced yes)
 		(effects
@@
 		)
 		(property "Intersheetrefs" "${INTERSHEET_REFS}"
-			(at 131.3078 50.8 0)
+			(at 225.3672 161.29 0)
 			(effects
 				(font
@@
 		)
 	)
-	(global_label "In_Vcc"
+	(global_label "display_supply"
+		(shape input)
+		(at 264.16 101.6 90)
+		(effects
+			(font
+				(size 1.27 1.27)
+			)
+			(justify left)
+		)
+		(property "Intersheetrefs" "${INTERSHEET_REFS}"
+			(at 264.16 101.6 0)
+			(effects
+				(font
+					(size 1.27 1.27)
+				)
+				(hide yes)
+			)
+		)
+	)
+	(global_label "C_BAT+"
+		(shape input)
+		(at 121.92 50.8 0)
+		(fields_autoplaced yes)
+		(effects
+			(font
+				(size 1.27 1.27)
+			)
+			(justify left)
+		)
+		(property "Intersheetrefs" "${INTERSHEET_REFS}"
+			(at 131.3872 50.8 0)
+			(effects
+				(font
+					(size 1.27 1.27)
+				)
+				(justify left)
+				(hide yes)
+			)
+		)
+	)
+	(global_label "display_supply"
 		(shape input)
 		(at 93.98 100.33 180)
@@
 		)
 	)
-	(global_label "display_enable"
-		(shape input)
-		(at 95.25 124.46 180)
-		(effects
-			(font
-				(size 1.27 1.27)
-			)
-			(justify right)
-		)
-		(property "Intersheetrefs" "${INTERSHEET_REFS}"
-			(at 95.25 124.46 0)
-			(effects
-				(font
-					(size 1.27 1.27)
-				)
-				(hide yes)
-			)
-		)
-	)
 	(hierarchical_label "BMS_gnd"
 		(shape input)
@@
 	(hierarchical_label "5V"
 		(shape input)
-		(at 264.16 101.6 0)
+		(at 95.25 128.27 0)
 		(fields_autoplaced yes)
 		(effects

Commit message: Subimos todos los archivos de la v0.25
Parts:
- added JP2: SolderJumper_2_Open, Jumper:SolderJumper-2_P1.3mm_Open_RoundedPad1.0x1.5mm, symbol Jumper:SolderJumper_2_Open
- IC2: value TC1108-2.8VDBTR -> TC1108-3.3VDBTR
- renumbered R23 to R21, R24 to R22, R25 to R23, R26 to R24, R27 to R25, R28 to R26, R29 to R27, R30 to R28, R31 to R29
Connections:
- net BAT+ is gone; now on net C_BAT+: SW_Toggle1.1
- net 5V: now also JP2.2 (B)
- net display_supply: now also JP2.1 (A)
Other:
- note added: "BMS CIRCUIT: Charging: -TP4056 as a well-known charging IC, up to 500mA with a 2.1K PROG resistor. -We do not use NTC for the battery in order to save costs. Protection IC: -None. You must choose a battery with integrated PCM Boost Converter: -TPS61085TDGKR as main chip. -Toggle Switch. -5V fix output voltage. 1A maximum output current -New diode: B340LA-13-F USB type C -Type C connector. Power S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"
- note removed: "BMS CIRCUIT: Charging: -TP4056 as a well-known charging IC, up to 500mA with a 2.1K PROG resistor. -We do not use NTC for the battery in order to save costs. Protection IC: -None. You must choose a battery with integrated PCM Boost Converter: -TPS61085TDGKR as main chip. -Toggle Switch. -5V fix output voltage. 1A maximum output current -New diode: B340LA-13-F USB type C -Type C connector. -Only f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"
Changed lines of the file:
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@@
 	)
 	(junction
+		(at 95.25 125.73)
+		(diameter 0)
+		(color 0 0 0 0)
+	)
+	(junction
 		(at 186.69 134.62)
 		(diameter 0)
@@
 	)
 	(junction
+		(at 95.25 104.14)
+		(diameter 0)
+		(color 0 0 0 0)
+	)
+	(junction
 		(at 213.36 161.29)
 		(diameter 0)
@@
 	(wire
 		(pts
+			(xy 107.95 113.03) (xy 107.95 104.14)
+		)
+		(stroke
+			(width 0)
+			(type default)
+		)
+	)
+	(wire
+		(pts
 			(xy 158.75 105.41) (xy 196.85 105.41)
 		)
@@
 	(wire
 		(pts
+			(xy 95.25 125.73) (xy 95.25 128.27)
+		)
+		(stroke
+			(width 0)
+			(type default)
+		)
+	)
+	(wire
+		(pts
 			(xy 100.33 45.72) (xy 115.57 45.72)
 		)
@@
 		)
 	)
+	(wire
+		(pts
+			(xy 107.95 125.73) (xy 95.25 125.73)
+		)
+		(stroke
+			(width 0)
+			(type default)
+		)
+	)
 	(polyline
 		(pts
@@
 	(wire
 		(pts
+			(xy 95.25 104.14) (xy 95.25 109.22)
+		)
+		(stroke
+			(width 0)
+			(type default)
+		)
+	)
+	(wire
+		(pts
 			(xy 63.5 50.8) (xy 60.96 50.8)
 		)
@@
 	(wire
 		(pts
-			(xy 95.25 124.46) (xy 95.25 128.27)
+			(xy 95.25 124.46) (xy 95.25 125.73)
 		)
 		(stroke
@@
 	(wire
 		(pts
+			(xy 107.95 120.65) (xy 107.95 125.73)
+		)
+		(stroke
+			(width 0)
+			(type default)
+		)
+	)
+	(wire
+		(pts
 			(xy 240.03 33.02) (xy 241.3 33.02)
 		)
@@
 	(wire
 		(pts
-			(xy 95.25 100.33) (xy 95.25 109.22)
+			(xy 95.25 100.33) (xy 95.25 104.14)
 		)
 		(stroke
@@
 	(wire
 		(pts
+			(xy 107.95 104.14) (xy 95.25 104.14)
+		)
+		(stroke
+			(width 0)
+			(type default)
+		)
+	)
+	(wire
+		(pts
 			(xy 102.87 43.18) (xy 102.87 59.69)
 		)
@@
 		)
 	)
-	(text "BMS CIRCUIT:\nCharging:\n-TP4056 as a well-known charging IC, up to 500mA with a 2.1K PROG resistor.\n-We do not use NTC for the battery in order to save costs.\n\nProtection IC:\n-None. You must choose a battery with integrated PCM\n\nBoost Converter:\n-TPS61085TDGKR as main chip. \n-Toggle Switch.\n-5V fix output voltage. 1A maximum output current \n-New diode: B340LA-13-F\n\n\nUSB type C \n-Type C connector.\n-Only for charging\n\nPower Supply Main IC:\n- TC1108 - 2.8V\n- 300mA for the uc\n"
+	(text "BMS CIRCUIT:\nCharging:\n-TP4056 as a well-known charging IC, up to 500mA with a 2.1K PROG resistor.\n-We do not use NTC for the battery in order to save costs.\n\nProtection IC:\n-None. You must choose a battery with integrated PCM\n\nBoost Converter:\n-TPS61085TDGKR as main chip. \n-Toggle Switch.\n-5V fix output voltage. 1A maximum output current \n-New diode: B340LA-13-F\n\n\nUSB type C \n-Type C connector.\n\nPower Supply Main IC:\n- TC1108 - 3.3V\n- 300mA for the uc\n"
 		(exclude_from_sim no)
 		(at 22.098 187.452 0)
@@
 		)
 	)
-	(global_label "BAT+"
+	(global_label "C_BAT+"
 		(shape input)
 		(at 156.21 107.95 270)
@@
 		)
 		(property "Intersheetrefs" "${INTERSHEET_REFS}"
-			(at 156.21 115.1002 90)
+			(at 156.21 117.4172 90)
 			(effects
 				(font
@@
 		(on_board yes)
 		(dnp no)
-		(property "Reference" "R23"
+		(property "Reference" "R21"
 			(at 56.134 42.418 0)
 			(effects
@@
 			(project "PicBytesMicro"
 				(path "/36e2b0cc-9d11-4a29-a898-cd33b5ef9720/00000000-0000-0000-0000-00006009e6f5"
-					(reference "R23")
+					(reference "R21")
 					(unit 1)
 				)
@@
 		(on_board yes)
 		(dnp no)
-		(property "Reference" "R27"
+		(property "Reference" "R25"
 			(at 173.736 40.386 0)
 			(effects
@@
 			(project "PicBytesMicro"
 				(path "/36e2b0cc-9d11-4a29-a898-cd33b5ef9720/00000000-0000-0000-0000-00006009e6f5"
-					(reference "R27")
+					(reference "R25")
 					(unit 1)
 				)
@@
 		(on_board yes)
 		(dnp no)
-		(property "Reference" "R25"
+		(property "Reference" "R23"
 			(at 108.9152 58.42 0)
 			(effects
@@
 			(project "PicBytesMicro"
 				(path "/36e2b0cc-9d11-4a29-a898-cd33b5ef9720/00000000-0000-0000-0000-00006009e6f5"
-					(reference "R25")
+					(reference "R23")
 					(unit 1)
 				)
@@
 		(on_board yes)
 		(dnp no)
-		(property "Reference" "R26"
+		(property "Reference" "R24"
 			(at 117.8052 58.42 0)
 			(effects
@@
 			(project "PicBytesMicro"
 				(path "/36e2b0cc-9d11-4a29-a898-cd33b5ef9720/00000000-0000-0000-0000-00006009e6f5"
-					(reference "R26")
+					(reference "R24")
 					(unit 1)
 				)
@@
 		(on_board yes)
 		(dnp no)
-		(property "Reference" "R28"
+		(property "Reference" "R26"
 			(at 178.7652 114.4016 90)
 			(effects
@@
 			(project "PicBytesMicro"
 				(path "/36e2b0cc-9d11-4a29-a898-cd33b5ef9720/00000000-0000-0000-0000-00006009e6f5"
-					(reference "R28")
+					(reference "R26")
 					(unit 1)
 				)
@@
 		(on_board yes)
 		(dnp no)
-		(property "Reference" "R30"
+		(property "Reference" "R28"
 			(at 188.9252 115.6716 90)
 			(effects
@@
 			(project "PicBytesMicro"
 				(path "/36e2b0cc-9d11-4a29-a898-cd33b5ef9720/00000000-0000-0000-0000-00006009e6f5"
-					(reference "R30")
+					(reference "R28")
 					(unit 1)
 				)
@@
 			)
 		)
-		(property "Value" "TC1108-2.8VDBTR"
+		(property "Value" "TC1108-3.3VDBTR"
 			(at 153.67 156.8704 0)
 			(effects
@@
 		(on_board yes)
 		(dnp no)
-		(property "Reference" "R31"
+		(property "Reference" "R29"
 			(at 231.394 35.814 0)
 			(effects
@@
 			(project "PicBytesMicro"
 				(path "/36e2b0cc-9d11-4a29-a898-cd33b5ef9720/00000000-0000-0000-0000-00006009e6f5"
-					(reference "R31")
+					(reference "R29")
 					(unit 1)
 				)
@@
 		(on_board yes)
 		(dnp no)
-		(property "Reference" "R29"
+		(property "Reference" "R27"
 			(at 188.9252 87.7316 90)
 			(effects
@@
 			(project "PicBytesMicro"
 				(path "/36e2b0cc-9d11-4a29-a898-cd33b5ef9720/00000000-0000-0000-0000-00006009e6f5"
-					(reference "R29")
+					(reference "R27")
 					(unit 1)
 				)
@@
 	)
 	(symbol
+		(lib_id "Jumper:SolderJumper_2_Open")
+		(at 107.95 116.84 270)
+		(unit 1)
+		(exclude_from_sim no)
+		(in_bom yes)
+		(on_board yes)
+		(dnp no)
+		(property "Reference" "JP2"
+			(at 109.6772 115.6716 90)
+			(effects
+				(font
+					(size 1.27 1.27)
+				)
+				(justify left)
+			)
+		)
+		(property "Value" "SolderJumper_2_Open"
+			(at 104.14 106.68 0)
+			(effects
+				(font
+					(size 1.27 1.27)
+				)
+				(justify left)
+			)
+		)
+		(property "Footprint" "Jumper:SolderJumper-2_P1.3mm_Open_RoundedPad1.0x1.5mm"
+			(at 107.95 116.84 0)
+			(effects
+				(font
+					(size 1.27 1.27)
+				)
+				(hide yes)
+			)
+		)
+		(property "Datasheet" "~"
+			(at 107.95 116.84 0)
+			(effects
+				(font
+					(size 1.27 1.27)
+				)
+				(hide yes)
+			)
+		)
+		(property "Description" ""
+			(at 107.95 116.84 0)
+			(effects
+				(font
+					(size 1.27 1.27)
+				)
+				(hide yes)
+			)
+		)
+		(pin "1"
+		)
+		(pin "2"
+		)
+		(instances
+			(project "PixelBytesHost"
+				(path "/36e2b0cc-9d11-4a29-a898-cd33b5ef9720/00000000-0000-0000-0000-00006009e6f5"
+					(reference "JP2")
+					(unit 1)
+				)
+			)
+		)
+	)
+	(symbol
 		(lib_id "PicBytesMicro-rescue:KTR10EZPF4220-SamacSys_Parts")
 		(at 64.77 116.84 0)
@@
 		(on_board yes)
 		(dnp no)
-		(property "Reference" "R24"
+		(property "Reference" "R22"
 			(at 73.66 111.125 0)
 			(effects
@@
 			(project "PicBytesMicro"
 				(path "/36e2b0cc-9d11-4a29-a898-cd33b5ef9720/00000000-0000-0000-0000-00006009e6f5"
-					(reference "R24")
+					(reference "R22")
 					(unit 1)
 				)
