File: Kicad/PixelBytesHost/BatteryCharger.kicad_sch (KiCad schematic)
At the start: 28 parts, among them IC2 TC1108-3.3VDBTR, IC3 TPS61085TDGKR, J2 B2B-XH-2__LF__SN_, J3 629722000214, Q3 SMMBT5551LT1G

Commit message: no message
Parts:
- J3: footprint 629722000214:629722000214 -> usb-c:629722000214
Changed lines of the file:
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@@
 			)
 		)
-		(property "Footprint" "629722000214:629722000214"
+		(property "Footprint" "usb-c:629722000214"
 			(at 209.55 40.64 0)
 			(effects
