File: Kicad/PixelBytesHost/BatteryCharger.kicad_sch (KiCad schematic)
At the start: 29 parts, among them IC2 TC1108-3.3VDBTR, IC3 TPS61085TDGKR, J2 B2B-XH-2__LF__SN_, J3 629722000214, Q3 PBSS5160T-QR

Commit message: no message
Parts:
- R22: value 6k8 -> 3K3
- R30: value 3k3 -> 2k
Changed lines of the file:
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@@
 			)
 		)
-		(property "Value" "6k8"
+		(property "Value" "3K3"
 			(at 64.77 113.4364 0)
 			(effects
@@
 			)
 		)
-		(property "Value" "3k3"
+		(property "Value" "2k"
 			(at 85.344 107.188 0)
 			(effects
