File: Kicad/PixelBytesHost/Dpad.kicad_sch (KiCad schematic)
At the start: 24 parts

Commit message: Subimos todos los archivos de la v0.25
Parts:
- renumbered R12 to R10, R13 to R11, R14 to R12, R15 to R13, R16 to R14, R17 to R15, R18 to R16, R19 to R17, R20 to R18, R21 to R19, R22 to R20, R11 to R9
Changed lines of the file:
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@@
 		(on_board yes)
 		(dnp no)
-		(property "Reference" "R21"
+		(property "Reference" "R19"
 			(at 236.22 103.505 0)
 			(effects
@@
 			(project "PicBytesMicro"
 				(path "/36e2b0cc-9d11-4a29-a898-cd33b5ef9720/00000000-0000-0000-0000-0000600718e8"
-					(reference "R21")
+					(reference "R19")
 					(unit 1)
 				)
@@
 		(on_board yes)
 		(dnp no)
-		(property "Reference" "R22"
+		(property "Reference" "R20"
 			(at 245.11 67.31 0)
 			(effects
@@
 			(project "PicBytesMicro"
 				(path "/36e2b0cc-9d11-4a29-a898-cd33b5ef9720/00000000-0000-0000-0000-0000600718e8"
-					(reference "R22")
+					(reference "R20")
 					(unit 1)
 				)
@@
 		(on_board yes)
 		(dnp no)
-		(property "Reference" "R18"
+		(property "Reference" "R16"
 			(at 161.29 86.995 0)
 			(effects
@@
 			(project "PicBytesMicro"
 				(path "/36e2b0cc-9d11-4a29-a898-cd33b5ef9720/00000000-0000-0000-0000-0000600718e8"
-					(reference "R18")
+					(reference "R16")
 					(unit 1)
 				)
@@
 		(on_board yes)
 		(dnp no)
-		(property "Reference" "R15"
+		(property "Reference" "R13"
 			(at 118.11 61.468 0)
 			(effects
@@
 			(project "PicBytesMicro"
 				(path "/36e2b0cc-9d11-4a29-a898-cd33b5ef9720/00000000-0000-0000-0000-0000600718e8"
-					(reference "R15")
+					(reference "R13")
 					(unit 1)
 				)
@@
 		(on_board yes)
 		(dnp no)
-		(property "Reference" "R12"
+		(property "Reference" "R10"
 			(at 81.28 88.9 0)
 			(effects
@@
 			(project "PicBytesMicro"
 				(path "/36e2b0cc-9d11-4a29-a898-cd33b5ef9720/00000000-0000-0000-0000-0000600718e8"
-					(reference "R12")
+					(reference "R10")
 					(unit 1)
 				)
@@
 		(on_board yes)
 		(dnp no)
-		(property "Reference" "R16"
+		(property "Reference" "R14"
 			(at 124.46 113.665 0)
 			(effects
@@
 			(project "PicBytesMicro"
 				(path "/36e2b0cc-9d11-4a29-a898-cd33b5ef9720/00000000-0000-0000-0000-0000600718e8"
-					(reference "R16")
+					(reference "R14")
 					(unit 1)
 				)
@@
 		(on_board yes)
 		(dnp no)
-		(property "Reference" "R19"
+		(property "Reference" "R17"
 			(at 209.55 95.885 0)
 			(effects
@@
 			(project "PicBytesMicro"
 				(path "/36e2b0cc-9d11-4a29-a898-cd33b5ef9720/00000000-0000-0000-0000-0000600718e8"
-					(reference "R19")
+					(reference "R17")
 					(unit 1)
 				)
@@
 		(on_board yes)
 		(dnp no)
-		(property "Reference" "R20"
+		(property "Reference" "R18"
 			(at 214.63 57.785 0)
 			(effects
@@
 			(project "PicBytesMicro"
 				(path "/36e2b0cc-9d11-4a29-a898-cd33b5ef9720/00000000-0000-0000-0000-0000600718e8"
-					(reference "R20")
+					(reference "R18")
 					(unit 1)
 				)
@@
 		(on_board yes)
 		(dnp no)
-		(property "Reference" "R13"
+		(property "Reference" "R11"
 			(at 100.33 106.045 0)
 			(effects
@@
 			(project "PicBytesMicro"
 				(path "/36e2b0cc-9d11-4a29-a898-cd33b5ef9720/00000000-0000-0000-0000-0000600718e8"
-					(reference "R13")
+					(reference "R11")
 					(unit 1)
 				)
@@
 		(on_board yes)
 		(dnp no)
-		(property "Reference" "R14"
+		(property "Reference" "R12"
 			(at 93.98 64.135 0)
 			(effects
@@
 			(project "PicBytesMicro"
 				(path "/36e2b0cc-9d11-4a29-a898-cd33b5ef9720/00000000-0000-0000-0000-0000600718e8"
-					(reference "R14")
+					(reference "R12")
 					(unit 1)
 				)
@@
 		(on_board yes)
 		(dnp no)
-		(property "Reference" "R17"
+		(property "Reference" "R15"
 			(at 140.97 79.375 0)
 			(effects
@@
 			(project "PicBytesMicro"
 				(path "/36e2b0cc-9d11-4a29-a898-cd33b5ef9720/00000000-0000-0000-0000-0000600718e8"
-					(reference "R17")
+					(reference "R15")
 					(unit 1)
 				)
@@
 		(on_board yes)
 		(dnp no)
-		(property "Reference" "R11"
+		(property "Reference" "R9"
 			(at 52.07 82.55 0)
 			(effects
@@
 			(project "PicBytesMicro"
 				(path "/36e2b0cc-9d11-4a29-a898-cd33b5ef9720/00000000-0000-0000-0000-0000600718e8"
-					(reference "R11")
+					(reference "R9")
 					(unit 1)
 				)

Commit message: New Version PixelBytesHost
Parts:
- R10, R13, R14, R16, R19, R20: footprint RESC2012X65N -> Resistor_SMD:R_0805_2012Metric
- R11, R12, R15, R17, R18, R9: footprint User_lib:RESC2012X75N -> Resistor_SMD:R_0805_2012Metric
Changed lines of the file:
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@@
 			)
 		)
-		(property "Footprint" "RESC2012X65N"
+		(property "Footprint" "Resistor_SMD:R_0805_2012Metric"
 			(at 241.3 107.95 0)
 			(effects
@@
 			)
 		)
-		(property "Footprint" "RESC2012X65N"
+		(property "Footprint" "Resistor_SMD:R_0805_2012Metric"
 			(at 250.19 68.58 0)
 			(effects
@@
 			)
 		)
-		(property "Footprint" "RESC2012X65N"
+		(property "Footprint" "Resistor_SMD:R_0805_2012Metric"
 			(at 166.37 91.44 0)
 			(effects
@@
 			)
 		)
-		(property "Footprint" "RESC2012X65N"
+		(property "Footprint" "Resistor_SMD:R_0805_2012Metric"
 			(at 123.19 57.15 0)
 			(effects
@@
 			)
 		)
-		(property "Footprint" "RESC2012X65N"
+		(property "Footprint" "Resistor_SMD:R_0805_2012Metric"
 			(at 86.36 90.17 0)
 			(effects
@@
 			)
 		)
-		(property "Footprint" "RESC2012X65N"
+		(property "Footprint" "Resistor_SMD:R_0805_2012Metric"
 			(at 129.54 118.11 0)
 			(effects
@@
 			)
 		)
-		(property "Footprint" "User_lib:RESC2012X75N"
+		(property "Footprint" "Resistor_SMD:R_0805_2012Metric"
 			(at 214.63 100.33 0)
 			(effects
@@
 			)
 		)
-		(property "Footprint" "User_lib:RESC2012X75N"
+		(property "Footprint" "Resistor_SMD:R_0805_2012Metric"
 			(at 219.71 62.23 0)
 			(effects
@@
 			)
 		)
-		(property "Footprint" "User_lib:RESC2012X75N"
+		(property "Footprint" "Resistor_SMD:R_0805_2012Metric"
 			(at 105.41 110.49 0)
 			(effects
@@
 			)
 		)
-		(property "Footprint" "User_lib:RESC2012X75N"
+		(property "Footprint" "Resistor_SMD:R_0805_2012Metric"
 			(at 88.9 59.69 0)
 			(effects
@@
 			)
 		)
-		(property "Footprint" "User_lib:RESC2012X75N"
+		(property "Footprint" "Resistor_SMD:R_0805_2012Metric"
 			(at 146.05 83.82 0)
 			(effects
@@
 			)
 		)
-		(property "Footprint" "User_lib:RESC2012X75N"
+		(property "Footprint" "Resistor_SMD:R_0805_2012Metric"
 			(at 57.15 83.82 0)
 			(effects
