File: Kicad/PixelBytesHost/PixelBytesHost.kicad_sch (KiCad schematic)
At the start: 27 parts, among them IC1 2536030320001, J1 TC2030-MCP-NL, Q1 SMMBT5551LT1G, Q2 SMMBT5551LT1G, U1 Pixel Bytes Display, U2 STM32F103CBTx, Y1 CX2520DB12000D0GPSC1

Commit message: Demo binary for the board
Connections:
- net at U1.11 (Vdi_s5): now also U1.21 (Vdo_s6); no longer U1.17 (Vdo_s4)
- net at U1.12 (Vdo_s5): no longer U1.22 (Vdi_s6)
- new net: U1.17 (Vdo_s4), U1.22 (Vdi_s6)
Other:
- note added: "V0.25 CHANGELOG: -changed string 5 to 6 in the pixel display -Fixed BAT connector. -We now cut the 5V power supply"
Changed lines of the file:
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@@
 	)
 	(no_connect
-		(at 69.85 72.39)
+		(at 50.8 80.01)
 	)
 	(no_connect
@@
 		(at 332.74 111.76)
 	)
-	(wire
-		(pts
-			(xy 57.15 59.69) (xy 57.15 77.47)
-		)
-		(stroke
-			(width 0)
-			(type default)
-		)
-	)
 	(polyline
 		(pts
@@
 	(wire
 		(pts
-			(xy 68.58 80.01) (xy 68.58 74.93)
+			(xy 40.64 49.53) (xy 50.8 49.53)
 		)
 		(stroke
@@
 	(wire
 		(pts
-			(xy 40.64 49.53) (xy 50.8 49.53)
+			(xy 137.16 200.66) (xy 139.7 200.66)
 		)
 		(stroke
@@
 	(wire
 		(pts
-			(xy 137.16 200.66) (xy 139.7 200.66)
+			(xy 175.26 203.2) (xy 177.8 203.2)
 		)
 		(stroke
@@
 	(wire
 		(pts
-			(xy 175.26 203.2) (xy 177.8 203.2)
+			(xy 63.5 59.69) (xy 63.5 74.93)
 		)
 		(stroke
@@
 	(wire
 		(pts
+			(xy 63.5 74.93) (xy 69.85 74.93)
+		)
+		(stroke
+			(width 0)
+			(type default)
+		)
+	)
+	(wire
+		(pts
 			(xy 125.73 177.8) (xy 125.73 180.34)
 		)
@@
 	(wire
 		(pts
+			(xy 53.34 77.47) (xy 50.8 77.47)
+		)
+		(stroke
+			(width 0)
+			(type default)
+		)
+	)
+	(wire
+		(pts
 			(xy 185.42 123.19) (xy 181.61 123.19)
 		)
@@
 	(wire
 		(pts
+			(xy 53.34 72.39) (xy 53.34 77.47)
+		)
+		(stroke
+			(width 0)
+			(type default)
+		)
+	)
+	(wire
+		(pts
 			(xy 69.85 77.47) (xy 80.01 77.47)
 		)
@@
 	(wire
 		(pts
-			(xy 69.85 59.69) (xy 57.15 59.69)
-		)
-		(stroke
-			(width 0)
-			(type default)
-		)
-	)
-	(wire
-		(pts
 			(xy 200.66 123.19) (xy 200.66 124.46)
 		)
@@
 		)
 	)
-	(wire
-		(pts
-			(xy 57.15 77.47) (xy 50.8 77.47)
-		)
-		(stroke
-			(width 0)
-			(type default)
-		)
-	)
 	(polyline
 		(pts
@@
 	(wire
 		(pts
-			(xy 50.8 80.01) (xy 68.58 80.01)
-		)
-		(stroke
-			(width 0)
-			(type default)
-		)
-	)
-	(wire
-		(pts
 			(xy 132.08 60.96) (xy 129.54 60.96)
 		)
@@
 	(wire
 		(pts
+			(xy 69.85 59.69) (xy 63.5 59.69)
+		)
+		(stroke
+			(width 0)
+			(type default)
+		)
+	)
+	(wire
+		(pts
 			(xy 176.53 73.66) (xy 176.53 74.93)
 		)
@@
 	(wire
 		(pts
-			(xy 68.58 74.93) (xy 69.85 74.93)
+			(xy 50.8 67.31) (xy 68.58 67.31)
 		)
 		(stroke
@@
 	(wire
 		(pts
-			(xy 50.8 67.31) (xy 68.58 67.31)
+			(xy 176.53 45.72) (xy 176.53 48.26)
 		)
 		(stroke
@@
 	(wire
 		(pts
-			(xy 176.53 45.72) (xy 176.53 48.26)
+			(xy 160.02 229.87) (xy 162.56 229.87)
 		)
 		(stroke
@@
 	(wire
 		(pts
-			(xy 160.02 229.87) (xy 162.56 229.87)
+			(xy 255.27 78.74) (xy 259.08 78.74)
 		)
 		(stroke
@@
 	(wire
 		(pts
-			(xy 255.27 78.74) (xy 259.08 78.74)
+			(xy 218.44 43.18) (xy 215.9 43.18)
 		)
 		(stroke
@@
 	(wire
 		(pts
-			(xy 218.44 43.18) (xy 215.9 43.18)
+			(xy 185.42 205.74) (xy 185.42 208.28)
 		)
 		(stroke
@@
 	(wire
 		(pts
-			(xy 185.42 205.74) (xy 185.42 208.28)
+			(xy 53.34 72.39) (xy 69.85 72.39)
 		)
 		(stroke
@@
 		)
 	)
+	(text "V0.25 CHANGELOG:\n	-changed string 5 to 6 in the pixel display\n	-Fixed BAT connector.\n	-We now cut the 5V power supply"
+		(exclude_from_sim no)
+		(at 353.822 261.366 0)
+		(effects
+			(font
+				(size 1.27 1.27)
+			)
+		)
+	)
 	(text "Programming port using TAG-CONNECT to ST32"
 		(exclude_from_sim no)
@@
 		)
 		(instances
-			(project "PicBytesMicro"
+			(project "PixelBytesHost"
 				(path "/36e2b0cc-9d11-4a29-a898-cd33b5ef9720"
 					(page "3")
@@
 		)
 		(instances
-			(project "PicBytesMicro"
+			(project "PixelBytesHost"
 				(path "/36e2b0cc-9d11-4a29-a898-cd33b5ef9720"
 					(page "4")

Commit message: Subimos todos los archivos de la v0.25
Parts:
- removed R8, R9: 20, Resistor_SMD:R_0805_2012Metric, symbol OpenReflowPlate-rescue:ERJP6WF1303V-Library_Loader
- R8: renamed from R10; value 4k7 -> 1k5
Connections:
- net USB_D+: now also U2.33 (PA12)
- net USB_D-: now also U2.32 (PA11)
Other:
- note added: "V0.25 CHANGELOG: -Changed string 5 to 6 in the pixel display. -Fixed BAT connector. -We now cut the 5V power supply with a transistor. -Removed resistors from the USB lines."
- note removed: "V0.25 CHANGELOG: -changed string 5 to 6 in the pixel display -Fixed BAT connector. -We now cut the 5V power supply"

Commit message: Host HW 1.0 finished
Parts:
- removed Y1: CX2520DB12000D0GPSC1, CX2520DB12000D0GPSC1, symbol User_lib:CX2520DB12000D0GPSC1
- added Y1: 830055663, 830055663, symbol User:830055663
Connections:
- net OSC1: now also Y1.3 (CRYSTAL_2)
- net OSC2: now also Y1.1 (CRYSTAL_1)
- net Vgnd_main: now also Y1.2 (GND_&_LID_1), Y1.4 (GND_&_LID_2)
Other:
- note added: "V1 CHANGELOG: -8Mhz crystal for the bootloader compatibility. -New USB-C. (No cuts in PCB) -New Switch of the PCB V0.25 CHANGELOG: -Changed string 5 to 6 in the pixel display. -Fixed BAT connector. -We now cut the 5V power supply with a transistor. -Removed resistors from the USB lines."
- note removed: "V0.25 CHANGELOG: -Changed string 5 to 6 in the pixel display. -Fixed BAT connector. -We now cut the 5V power supply with a transistor. -Removed resistors from the USB lines."

Commit message: no message
Parts:
- R2, R3: value 20K -> 10K
Changed lines of the file:
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@@
 			)
 		)
-		(property "Value" "20K"
+		(property "Value" "10K"
 			(at 61.6712 177.673 90)
 			(effects
@@
 			)
 		)
-		(property "Value" "20K"
+		(property "Value" "10K"
 			(at 61.6712 200.533 90)
 			(effects

Commit message: New Version PixelBytesHost
Parts:
- added LED_green_bms2: LTST-C171GKT, LEDC2012X90N, symbol PicBytesMicro-rescue:LTST-C171GKT-SamacSys_Parts
- added R31: 10k, Resistor_SMD:R_0805_2012Metric, symbol OpenReflowPlate-rescue:ERJP6WF1303V-Library_Loader
- added R32: 1k, Resistor_SMD:R_0805_2012Metric, symbol OpenReflowPlate-rescue:ERJP6WF1303V-Library_Loader
- added S1: 434121025816, 434121050816, symbol User:434121025816
- C7, C8: footprint CAPC2012X145N -> Capacitor_SMD:C_0805_2012Metric
- R2, R3, R5, R6, R7: value 10K -> 10k
Connections:
- net Vgnd_main: now also LED_green_bms2.1 (K), R31.1
- net uc_enable_display: now also U2.45 (PB8); no longer U2.20 (PB2)
- net uc_supply: now also S1.2 (NO)
- net boot_led: now reaches U2.30 (PA9)
- net boot_led: now also R32.2
- new net: LED_green_bms2.2 (A), R32.1
- new net boot1: R31.2, S1.1 (COM), U2.20 (PB2)
- no-connect marks 19 -> 17
Other:
- note added: "bootloader peripherals"
