File: Kicad/PixelDisplay/PixelDisplay.kicad_pcb (KiCad board)
At the start: 4 copper layers, 36 x 47 mm, 253 parts, among them J1 Conn_01x04_Pin, J2 Conn_01x04_Pin, J3 Conn_01x04_Pin, J4 Conn_01x04_Pin, J5 Conn_01x04_Pin, J6 Conn_01x04_Pin

Commit message: no message
Parts:
- removed REF**: OSHW-Logo2_7.3x6mm_SilkScreen, Symbol:OSHW-Logo2_7.3x6mm_SilkScreen
- moved J1 0.25 mm to (134.3, 46.3)
- moved J2 0.25 mm to (170.8, 53.9)
- moved J3 0.25 mm to (134.3, 63.3)
- moved J4 0.25 mm to (170.9, 70.8)
- moved J5 0.25 mm to (170.8, 91.2)
- moved J6 0.25 mm to (134.3, 83.5)
Routing:
- net Vss_str4: track 145.0 -> 146.9 mm
- net Vss_str3: track 142.1 -> 143.7 mm
- net Vss_str5: track 142.9 -> 144.3 mm
- net Vss_str2: track 142.3 -> 143.5 mm
- net Vdd_str3: track 153.5 -> 154.0 mm
Other:
- board size 36 x 47 mm -> 36.5 x 47.2 mm
